Commit message: make setting acm part of the grasp planner

File: robots/suction_hand.xacro (robot description, xacro)
@@ -13,13 +13,13 @@
         <origin xyz="0.0 0.0 0.055" rpy="0.0 0.0 0.0" />
         <geometry>
-          <box size="0.25 0.13 0.1"/>
+          <box size="0.0625 0.0625 0.1"/>
         </geometry>
       </visual>
-      <collision>
-        <origin xyz="0.0 0.0 0.055" rpy="0.0 0.0 0.0" />
+      <visual>
+        <origin xyz="0.0 0.0 0.125" rpy="0.0 0.0 0.0" />
         <geometry>
-          <box size="0.25 0.13 0.1"/>
+          <box size="0.25 0.13 0.05"/>
         </geometry>
-      </collision>
+      </visual>
     </link>
     <link name="tool_center_point" />
@@ -27,5 +27,5 @@
       <parent link="${ns}_hand"/>
       <child link = "tool_center_point" />
-      <origin xyz="0.0 0.0 0.105" rpy="0.0 0.0 0.0" />
+      <origin xyz="0.0 0.0 0.15" rpy="0.0 0.0 0.0" />
     </joint>
   </xacro:macro>

Commit message: Add collision for suction hand (smaller than visual)

File: robots/suction_hand.xacro (robot description, xacro)
@@ -22,4 +22,16 @@
         </geometry>
       </visual>
+      <collision>
+        <origin xyz="0.0 0.0 0.055" rpy="0.0 0.0 0.0" />
+        <geometry>
+          <box size="0.0625 0.0625 0.1"/>
+        </geometry>
+      </collision>
+      <collision>
+        <origin xyz="0.0 0.0 0.11" rpy="0.0 0.0 0.0" />
+        <geometry>
+          <box size="0.25 0.13 0.02"/>
+        </geometry>
+      </collision>
     </link>
     <link name="tool_center_point" />
