Commit message: Adaptions for recent franka_description + panda_moveit_config

File: robots/panda_arm_suction_hand.srdf.xacro (robot description, xacro)
@@ -5,7 +5,6 @@
 -->
 <robot xmlns:xacro="http://www.ros.org/wiki/xacro" name="panda">
-  <xacro:include filename="$(find panda_moveit_config)/config/panda_arm.xacro" />
-  <xacro:panda_arm />
-  <group name="hand">
+  <xacro:include filename="$(find panda_moveit_config)/config/panda.srdf.xacro"/>
+  <group name="panda_hand">
     <link name="panda_hand" />
     <link name="tool_center_point" />
@@ -18,5 +17,5 @@
   <group name="panda_arm_hand">
     <group name="panda_arm" />
-    <group name="hand" />
+    <group name="panda_hand"/>
   </group>
   <!--GROUP STATES: Purpose: Define a named state for a particular group, in terms of joint values. This is useful to define states like 'folded arms'-->
@@ -40,5 +39,5 @@
   </group_state>
   <!--END EFFECTOR: Purpose: Represent information about an end effector.-->
-  <end_effector name="hand" parent_link="panda_link8" group="hand" parent_group="panda_arm" />
+  <end_effector name="panda_hand" parent_link="panda_link8" group="panda_hand" parent_group="panda_arm"/>
   <!--DISABLE COLLISIONS: By default it is assumed that any link of the robot could potentially come into collision with any other link in the robot. This tag disables collision checking between a specified pair of links. -->
   <disable_collisions link1="panda_hand" link2="panda_link3" reason="Never" />

File: robots/panda_arm_suction_hand.urdf.xacro (robot description, xacro)
@@ -1,7 +1,6 @@
 <?xml version="1.0" encoding="utf-8"?>
 <robot xmlns:xacro="http://www.ros.org/wiki/xacro" name="panda">
-  <xacro:include filename="$(find franka_description)/robots/panda_arm.xacro"/>
+  <xacro:include filename="$(find franka_description)/robots/panda/panda.urdf.xacro"/>
   <xacro:include filename="$(find moveit_grasps)/robots/suction_hand.xacro"/>
-  <xacro:panda_arm />
-  <xacro:suction_hand ns="panda" rpy="0 0 ${-pi/4}" connected_to="panda_link8"/>
+  <xacro:suction_hand ns="$(arg arm_id)" rpy="0 0 ${-pi/4}" connected_to="$(arg arm_id)_link8"/>
 </robot>

File: robots/panda_arm_two_finger_hand.srdf.xacro (robot description, xacro)
@@ -5,8 +5,6 @@
 -->
 <robot xmlns:xacro="http://www.ros.org/wiki/xacro" name="panda">
-  <xacro:include filename="$(find panda_moveit_config)/config/panda_arm.xacro" />
-  <xacro:include filename="$(find panda_moveit_config)/config/hand.xacro" />
-  <xacro:panda_arm />
-  <xacro:hand />
+  <xacro:arg name="hand" default="true"/>
+  <xacro:include filename="$(find panda_moveit_config)/config/panda.srdf.xacro"/>
   <!--GROUPS: Representation of a set of joints and links. This can be useful for specifying DOF to plan for, defining arms, end effectors, etc-->
   <!--LINKS: When a link is specified, the parent joint of that link (if it exists) is automatically included-->
@@ -15,9 +13,9 @@
   <!--SUBGROUPS: Groups can also be formed by referencing to already defined group names-->
   <group name="panda_arm_hand">
-    <group name="panda_arm" />
-    <group name="hand" />
+    <group name="panda_manipulator"/>
+    <group name="panda_hand"/>
   </group>
   <!--GROUP STATES: Purpose: Define a named state for a particular group, in terms of joint values. This is useful to define states like 'folded arms'-->
-  <group_state name="ready" group="panda_arm_hand">
+  <group_state name="ready" group="panda_arm">
     <joint name="panda_joint1" value="0" />
     <joint name="panda_joint2" value="-0.785" />
@@ -28,5 +26,5 @@
     <joint name="panda_joint7" value="0.785" />
   </group_state>
-  <group_state name="extended" group="panda_arm_hand">
+  <group_state name="extended" group="panda_arm">
     <joint name="panda_joint1" value="0" />
     <joint name="panda_joint2" value="0" />
@@ -37,26 +35,13 @@
     <joint name="panda_joint7" value="0.785" />
   </group_state>
-  <group_state name="open" group="hand">
+  <group_state name="open" group="panda_hand">
     <joint name="panda_finger_joint1" value="0.035" />
     <joint name="panda_finger_joint2" value="0.035" />
   </group_state>
-  <group_state name="close" group="hand">
+  <group_state name="close" group="panda_hand">
     <joint name="panda_finger_joint1" value="0" />
     <joint name="panda_finger_joint2" value="0" />
   </group_state>
   <!--END EFFECTOR: Purpose: Represent information about an end effector.-->
-  <end_effector name="hand" parent_link="panda_link8" group="hand" parent_group="panda_arm" />
-  <!--DISABLE COLLISIONS: By default it is assumed that any link of the robot could potentially come into collision with any other link in the robot. This tag disables collision checking between a specified pair of links. -->
-  <disable_collisions link1="panda_hand" link2="panda_link3" reason="Never" />
-  <disable_collisions link1="panda_hand" link2="panda_link4" reason="Never" />
-  <disable_collisions link1="panda_hand" link2="panda_link6" reason="Never" />
-  <disable_collisions link1="panda_hand" link2="panda_link7" reason="Adjacent" />
-  <disable_collisions link1="panda_leftfinger" link2="panda_link3" reason="Never" />
-  <disable_collisions link1="panda_leftfinger" link2="panda_link4" reason="Never" />
-  <disable_collisions link1="panda_leftfinger" link2="panda_link6" reason="Never" />
-  <disable_collisions link1="panda_leftfinger" link2="panda_link7" reason="Never" />
-  <disable_collisions link1="panda_link3" link2="panda_rightfinger" reason="Never" />
-  <disable_collisions link1="panda_link4" link2="panda_rightfinger" reason="Never" />
-  <disable_collisions link1="panda_link6" link2="panda_rightfinger" reason="Never" />
-  <disable_collisions link1="panda_link7" link2="panda_rightfinger" reason="Never" />
+  <end_effector name="panda_hand" parent_link="panda_link8" group="panda_hand" parent_group="panda_arm"/>
 </robot>

File: robots/panda_arm_two_finger_hand.urdf.xacro (robot description, xacro)
@@ -1,7 +1,10 @@
 <?xml version="1.0" encoding="utf-8"?>
 <robot xmlns:xacro="http://www.ros.org/wiki/xacro" name="panda">
-  <xacro:include filename="$(find franka_description)/robots/panda_arm.xacro"/>
-  <xacro:include filename="$(find moveit_grasps)/robots/two_finger_hand.xacro"/>
-  <xacro:panda_arm />
-  <xacro:two_finger_hand ns="panda" rpy="0 0 ${-pi/4}" connected_to="panda_link8"/>
+  <xacro:arg name="hand" default="true"/>
+  <xacro:include filename="$(find franka_description)/robots/panda/panda.urdf.xacro"/>
+  <link name="tool_center_point"/>
+  <joint name="tool_center_point_joint" type="fixed">
+    <parent link="$(arg arm_id)_hand_tcp"/>
+    <child link="tool_center_point"/>
+  </joint>
 </robot>
